File: current_monitor_v1-1.brd (EAGLE design)
At the start: 81 x 54.4 mm, 43 parts, among them IC1 LM4558D, SW1 RESET, SW2 Display, SW3 Display, U1 ATMEGA32U4-XUAU, Y1 16MHz

Commit message: submitted to fab 11/3/14 -- fixed agnd and usb drill sizes
Parts:
- added JP2: M01PTH, SparkFun-Connectors:1X01
- U$12: value USB-MICRO-B-EVT -> USB-MICRO-B-UNIVERSAL; device _usb_micro_b:USB-MICRO-B-UNIVERSAL-SOLID-FOOTS -> _usb_micro_b:USB-MICRO-B-UNIVERSAL
Connections:
- net N$1: now also IC1.5; no longer IC1.6
- net N$2: now also IC1.2; no longer IC1.3
- net N$3: now also IC1.6; no longer IC1.5
- net N$6: now also IC1.3; no longer IC1.2
Routing:
- net N$1: track 39.6 -> 35.2 mm, vias 2 -> 4
- net N$3: track 15.2 -> 18.2 mm
- net N$6: track 26.4 -> 24.5 mm
- net N$2: track 8.73 -> 10.4 mm
